File: my-keyboard.kicad_pcb (KiCad board)
At the start: 2 copper layers, 161.9 x 58.7 mm, 24 parts, among them SW1 SW_Push, U1 ATmega32U4-AU, Y1 16MHz

Commit message: wires and pcb
Parts:
- added D10: D_Small, Diode_SMD:D_SOD-123, B.Cu at (131.0, 169.9)
- added D11: D_Small, Diode_SMD:D_SOD-123, B.Cu at (123.0, 208.0)
- added D12: D_Small, Diode_SMD:D_SOD-123, B.Cu at (134.9, 112.7)
- added D13: D_Small, Diode_SMD:D_SOD-123, B.Cu at (134.9, 131.8)
- added D14: D_Small, Diode_SMD:D_SOD-123, B.Cu at (144.5, 150.8)
- added D15: D_Small, Diode_SMD:D_SOD-123, B.Cu at (149.2, 169.9)
- added D16: D_Small, Diode_SMD:D_SOD-123, B.Cu at (139.7, 188.9)
- added D17: D_Small, Diode_SMD:D_SOD-123, B.Cu at (146.8, 208.0)
- added D18: D_Small, Diode_SMD:D_SOD-123, B.Cu at (154.0, 112.7)
- added D19: D_Small, Diode_SMD:D_SOD-123, B.Cu at (154.0, 131.8)
- added D20: D_Small, Diode_SMD:D_SOD-123, B.Cu at (163.5, 150.8)
- added D21: D_Small, Diode_SMD:D_SOD-123, B.Cu at (168.3, 169.9)
- added D22: D_Small, Diode_SMD:D_SOD-123, B.Cu at (158.8, 188.9)
- added D23: D_Small, Diode_SMD:D_SOD-123, B.Cu at (173.0, 112.7)
- added D24: D_Small, Diode_SMD:D_SOD-123, B.Cu at (173.0, 131.8)
- added D25: D_Small, Diode_SMD:D_SOD-123, B.Cu at (182.6, 150.8)
- added D26: D_Small, Diode_SMD:D_SOD-123, B.Cu at (187.3, 169.9)
- added D27: D_Small, Diode_SMD:D_SOD-123, B.Cu at (177.8, 188.9)
- added D28: D_Small, Diode_SMD:D_SOD-123, B.Cu at (192.1, 112.7)
- added D29: D_Small, Diode_SMD:D_SOD-123, B.Cu at (192.1, 131.8)
- added D30: D_Small, Diode_SMD:D_SOD-123, B.Cu at (201.6, 150.8)
- added D31: D_Small, Diode_SMD:D_SOD-123, B.Cu at (206.4, 169.9)
- added D32: D_Small, Diode_SMD:D_SOD-123, B.Cu at (196.8, 188.9)
- added D33: D_Small, Diode_SMD:D_SOD-123, B.Cu at (211.1, 112.7)
- added D34: D_Small, Diode_SMD:D_SOD-123, B.Cu at (211.1, 131.8)
- added D35: D_Small, Diode_SMD:D_SOD-123, B.Cu at (220.7, 150.8)
- added D36: D_Small, Diode_SMD:D_SOD-123, B.Cu at (225.4, 169.9)
- added D37: D_Small, Diode_SMD:D_SOD-123, B.Cu at (215.9, 188.9)
- added D38: D_Small, Diode_SMD:D_SOD-123, B.Cu at (225.4, 208.0)
- added D39: D_Small, Diode_SMD:D_SOD-123, B.Cu at (230.2, 112.7)
- added D40: D_Small, Diode_SMD:D_SOD-123, B.Cu at (230.2, 131.8)
- added D41: D_Small, Diode_SMD:D_SOD-123, B.Cu at (239.7, 150.8)
- added D42: D_Small, Diode_SMD:D_SOD-123, B.Cu at (244.5, 169.9)
- added D43: D_Small, Diode_SMD:D_SOD-123, B.Cu at (234.9, 188.9)
- added D44: D_Small, Diode_SMD:D_SOD-123, B.Cu at (249.2, 112.7)
- added D45: D_Small, Diode_SMD:D_SOD-123, B.Cu at (249.2, 131.8)
- added D46: D_Small, Diode_SMD:D_SOD-123, B.Cu at (258.8, 150.8)
- added D47: D_Small, Diode_SMD:D_SOD-123, B.Cu at (263.5, 169.9)
- added D48: D_Small, Diode_SMD:D_SOD-123, B.Cu at (254.0, 188.9)
- added D49: D_Small, Diode_SMD:D_SOD-123, B.Cu at (268.3, 112.7)
- added D5: D_Small, Diode_SMD:D_SOD-123, B.Cu at (101.6, 150.8)
- added D50: D_Small, Diode_SMD:D_SOD-123, B.Cu at (268.3, 131.8)
- added D51: D_Small, Diode_SMD:D_SOD-123, B.Cu at (277.8, 150.8)
- added D52: D_Small, Diode_SMD:D_SOD-123, B.Cu at (282.6, 169.9)
- added D53: D_Small, Diode_SMD:D_SOD-123, B.Cu at (273.1, 188.9)
- added D54: D_Small, Diode_SMD:D_SOD-123, B.Cu at (287.3, 112.8)
- added D55: D_Small, Diode_SMD:D_SOD-123, B.Cu at (287.3, 131.8)
- added D56: D_Small, Diode_SMD:D_SOD-123, B.Cu at (296.9, 150.8)
- added D57: D_Small, Diode_SMD:D_SOD-123, B.Cu at (301.6, 169.9)
- added D58: D_Small, Diode_SMD:D_SOD-123, B.Cu at (292.1, 188.9)
- added D59: D_Small, Diode_SMD:D_SOD-123, B.Cu at (287.3, 208.0)
- added D6: D_Small, Diode_SMD:D_SOD-123, B.Cu at (104.0, 169.9)
- added D60: D_Small, Diode_SMD:D_SOD-123, B.Cu at (306.4, 112.7)
- added D61: D_Small, Diode_SMD:D_SOD-123, B.Cu at (306.4, 131.8)
- added D62: D_Small, Diode_SMD:D_SOD-123, B.Cu at (315.9, 150.8)
- added D63: D_Small, Diode_SMD:D_SOD-123, B.Cu at (320.7, 169.9)
- added D64: D_Small, Diode_SMD:D_SOD-123, B.Cu at (311.1, 188.9)
- added D65: D_Small, Diode_SMD:D_SOD-123, B.Cu at (306.4, 208.0)
- added D66: D_Small, Diode_SMD:D_SOD-123, B.Cu at (325.4, 112.7)
- added D67: D_Small, Diode_SMD:D_SOD-123, B.Cu at (325.4, 131.8)
- added D68: D_Small, Diode_SMD:D_SOD-123, B.Cu at (335.0, 150.8)
- added D69: D_Small, Diode_SMD:D_SOD-123, B.Cu at (351.6, 169.9)
- added D7: D_Small, Diode_SMD:D_SOD-123, B.Cu at (108.7, 188.9)
- added D70: D_Small, Diode_SMD:D_SOD-123, B.Cu at (337.3, 188.9)
- added D71: D_Small, Diode_SMD:D_SOD-123, B.Cu at (325.4, 208.0)
- added D72: D_Small, Diode_SMD:D_SOD-123, B.Cu at (344.5, 112.7)
- added D73: D_Small, Diode_SMD:D_SOD-123, B.Cu at (354.0, 131.8)
- added D74: D_Small, Diode_SMD:D_SOD-123, B.Cu at (358.8, 150.8)
- added D76: D_Small, Diode_SMD:D_SOD-123, B.Cu at (344.5, 208.0)
- added D77: D_Small, Diode_SMD:D_SOD-123, B.Cu at (363.5, 112.7)
- added D78: D_Small, Diode_SMD:D_SOD-123, B.Cu at (363.5, 188.9)
- added D79: D_Small, Diode_SMD:D_SOD-123, B.Cu at (363.5, 208.0)
- added D8: D_Small, Diode_SMD:D_SOD-123, B.Cu at (99.2, 208.0)
- added D80: D_Small, Diode_SMD:D_SOD-123, B.Cu at (382.6, 112.7)
- added D81: D_Small, Diode_SMD:D_SOD-123, B.Cu at (382.6, 131.8)
- added D82: D_Small, Diode_SMD:D_SOD-123, B.Cu at (382.6, 150.8)
- added D83: D_Small, Diode_SMD:D_SOD-123, B.Cu at (382.6, 169.9)
- added D84: D_Small, Diode_SMD:D_SOD-123, B.Cu at (382.6, 188.9)
- added D85: D_Small, Diode_SMD:D_SOD-123, B.Cu at (382.6, 208.0)
- added D9: D_Small, Diode_SMD:D_SOD-123, B.Cu at (125.4, 150.8)
- added J1: AVR-ISP-6, Connector_PinHeader_1.00mm:PinHeader_2x03_P1.00mm_Horizontal, F.Cu at (73.0, 108.7)
- added MX0-2: F2, MX_Alps_Hybrid:MX-1U-NoLED, F.Cu at (127.0, 112.7)
- added MX0-3: F3, MX_Alps_Hybrid:MX-1U-NoLED, F.Cu at (146.1, 112.7)
- added MX0-4: F4, MX_Alps_Hybrid:MX-1U-NoLED, F.Cu at (165.1, 112.7)
- added MX0-5: F5, MX_Alps_Hybrid:MX-1U-NoLED, F.Cu at (184.2, 112.7)
- added MX1-10: 0, MX_Alps_Hybrid:MX-1U-NoLED, F.Cu at (279.4, 131.8)
- added MX1-11: -, MX_Alps_Hybrid:MX-1U-NoLED, F.Cu at (298.4, 131.8)
- added MX1-12: =, MX_Alps_Hybrid:MX-1U-NoLED, F.Cu at (317.5, 131.8)
- added MX1-13: Backspace, MX_Alps_Hybrid:MX-2U-NoLED, F.Cu at (346.1, 131.8)
- added MX1-15: PgUp, MX_Alps_Hybrid:MX-1U-NoLED, F.Cu at (374.6, 131.8)
- added MX1-2: 2, MX_Alps_Hybrid:MX-1U-NoLED, F.Cu at (127.0, 131.8)
- added MX1-3: 3, MX_Alps_Hybrid:MX-1U-NoLED, F.Cu at (146.1, 131.8)
- added MX1-4: 4, MX_Alps_Hybrid:MX-1U-NoLED, F.Cu at (165.1, 131.8)
- added MX1-5: 5, MX_Alps_Hybrid:MX-1U-NoLED, F.Cu at (184.2, 131.8)
- added MX1-6: 6, MX_Alps_Hybrid:MX-1U-NoLED, F.Cu at (203.2, 131.8)
- added MX1-7: 7, MX_Alps_Hybrid:MX-1U-NoLED, F.Cu at (222.2, 131.8)
- added MX1-8: 8, MX_Alps_Hybrid:MX-1U-NoLED, F.Cu at (241.3, 131.8)
- added MX1-9: 9, MX_Alps_Hybrid:MX-1U-NoLED, F.Cu at (260.4, 131.8)
- added MX10-0: F10, MX_Alps_Hybrid:MX-1U-NoLED, F.Cu at (279.4, 112.7)
- added MX11-0: F11, MX_Alps_Hybrid:MX-1U-NoLED, F.Cu at (298.4, 112.7)
- added MX12-0: F12, MX_Alps_Hybrid:MX-1U-NoLED, F.Cu at (317.5, 112.7)
- added MX13-0: PrtSc, MX_Alps_Hybrid:MX-1U-NoLED, F.Cu at (336.6, 112.7)
- added MX14-0: Scroll Lock, MX_Alps_Hybrid:MX-1U-NoLED, F.Cu at (355.6, 112.7)
- added MX15-0: Del, MX_Alps_Hybrid:MX-1U-NoLED, F.Cu at (374.6, 112.7)
- added MX2-0: Tab, MX_Alps_Hybrid:MX-1.5U-NoLED, F.Cu at (93.7, 150.8)
- added MX2-1: Q, MX_Alps_Hybrid:MX-1U-NoLED, F.Cu at (117.5, 150.8)
- added MX2-10: P, MX_Alps_Hybrid:MX-1U-NoLED, F.Cu at (288.9, 150.8)
- added MX2-11: [, MX_Alps_Hybrid:MX-1U-NoLED, F.Cu at (308.0, 150.8)
- added MX2-12: ], MX_Alps_Hybrid:MX-1U-NoLED, F.Cu at (327.0, 150.8)
- added MX2-13: \, MX_Alps_Hybrid:MX-1.5U-NoLED, F.Cu at (350.8, 150.8)
- added MX2-15: PgDn, MX_Alps_Hybrid:MX-1U-NoLED, F.Cu at (374.6, 150.8)
- added MX2-2: W, MX_Alps_Hybrid:MX-1U-NoLED, F.Cu at (136.5, 150.8)
- added MX2-3: E, MX_Alps_Hybrid:MX-1U-NoLED, F.Cu at (155.6, 150.8)
- added MX2-4: R, MX_Alps_Hybrid:MX-1U-NoLED, F.Cu at (174.6, 150.8)
- added MX2-5: T, MX_Alps_Hybrid:MX-1U-NoLED, F.Cu at (193.7, 150.8)
- added MX2-6: Y, MX_Alps_Hybrid:MX-1U-NoLED, F.Cu at (212.7, 150.8)
- added MX2-7: U, MX_Alps_Hybrid:MX-1U-NoLED, F.Cu at (231.8, 150.8)
- added MX2-8: I, MX_Alps_Hybrid:MX-1U-NoLED, F.Cu at (250.8, 150.8)
- added MX2-9: O, MX_Alps_Hybrid:MX-1U-NoLED, F.Cu at (269.9, 150.8)
- added MX3-0: Caps Lock, MX_Alps_Hybrid:MX-1.75U, F.Cu at (96.0, 169.9)
- added MX3-1: A, MX_Alps_Hybrid:MX-1U-NoLED, F.Cu at (122.2, 169.9)
- added MX3-10: ;, MX_Alps_Hybrid:MX-1U-NoLED, F.Cu at (293.7, 169.9)
- added MX3-11: ', MX_Alps_Hybrid:MX-1U-NoLED, F.Cu at (312.7, 169.9)
- added MX3-12: return, MX_Alps_Hybrid:MX-2.25U-NoLED, F.Cu at (343.7, 169.9)
- added MX3-15: Home, MX_Alps_Hybrid:MX-1U-NoLED, F.Cu at (374.6, 169.9)
- added MX3-2: S, MX_Alps_Hybrid:MX-1U-NoLED, F.Cu at (141.3, 169.9)
- added MX3-3: D, MX_Alps_Hybrid:MX-1U-NoLED, F.Cu at (160.3, 169.9)
- added MX3-4: F, MX_Alps_Hybrid:MX-1U-NoLED, F.Cu at (179.4, 169.9)
- added MX3-5: G, MX_Alps_Hybrid:MX-1U-NoLED, F.Cu at (198.4, 169.9)
- added MX3-6: H, MX_Alps_Hybrid:MX-1U-NoLED, F.Cu at (217.5, 169.9)
- added MX3-7: J, MX_Alps_Hybrid:MX-1U-NoLED, F.Cu at (236.5, 169.9)
- added MX3-8: K, MX_Alps_Hybrid:MX-1U-NoLED, F.Cu at (255.6, 169.9)
- added MX3-9: L, MX_Alps_Hybrid:MX-1U-NoLED, F.Cu at (274.6, 169.9)
- added MX4-0: Shift, MX_Alps_Hybrid:MX-2.25U-NoLED, F.Cu at (100.8, 188.9)
- added MX4-10: ., MX_Alps_Hybrid:MX-1U-NoLED, F.Cu at (284.2, 188.9)
- added MX4-11: /, MX_Alps_Hybrid:MX-1U-NoLED, F.Cu at (303.2, 188.9)
- added MX4-12: Shift, MX_Alps_Hybrid:MX-1.75U-NoLED, F.Cu at (329.4, 188.9)
- added MX4-13: Up, MX_Alps_Hybrid:MX-1U-NoLED, F.Cu at (355.6, 188.9)
- added MX4-14: End, MX_Alps_Hybrid:MX-1U-NoLED, F.Cu at (374.6, 188.9)
- added MX4-2: Z, MX_Alps_Hybrid:MX-1U-NoLED, F.Cu at (131.8, 188.9)
- added MX4-3: X, MX_Alps_Hybrid:MX-1U-NoLED, F.Cu at (150.8, 188.9)
- added MX4-4: C, MX_Alps_Hybrid:MX-1U-NoLED, F.Cu at (169.9, 188.9)
- added MX4-5: V, MX_Alps_Hybrid:MX-1U-NoLED, F.Cu at (188.9, 188.9)
- added MX4-6: B, MX_Alps_Hybrid:MX-1U-NoLED, F.Cu at (208.0, 188.9)
- added MX4-7: N, MX_Alps_Hybrid:MX-1U-NoLED, F.Cu at (227.0, 188.9)
- added MX4-8: M, MX_Alps_Hybrid:MX-1U-NoLED, F.Cu at (246.1, 188.9)
- added MX4-9: ,, MX_Alps_Hybrid:MX-1U-NoLED, F.Cu at (265.1, 188.9)
- added MX5-0: LCtrl, MX_Alps_Hybrid:MX-1.25U-NoLED, F.Cu at (91.3, 208.0)
- added MX5-1: LMeta, MX_Alps_Hybrid:MX-1.25U-NoLED, F.Cu at (115.1, 208.0)
- added MX5-10: Menu, MX_Alps_Hybrid:MX-1U-NoLED, F.Cu at (298.4, 208.0)
- added MX5-11: RCtrl, MX_Alps_Hybrid:MX-1U-NoLED, F.Cu at (317.5, 208.0)
- added MX5-12: Left, MX_Alps_Hybrid:MX-1U-NoLED, F.Cu at (336.6, 208.0)
- added MX5-13: Down, MX_Alps_Hybrid:MX-1U-NoLED, F.Cu at (355.6, 208.0)
- added MX5-14: Right, MX_Alps_Hybrid:MX-1U-NoLED, F.Cu at (374.6, 208.0)
- added MX5-2: Alt, MX_Alps_Hybrid:MX-1.25U-NoLED, F.Cu at (138.9, 208.0)
- added MX5-6: Space, MX_Alps_Hybrid:MX-6U-NoLED, F.Cu at (208.0, 208.0)
- added MX5-9: RMeta, MX_Alps_Hybrid:MX-1.25U-NoLED, F.Cu at (277.0, 208.0)
- added MX6-0: F6, MX_Alps_Hybrid:MX-1U-NoLED, F.Cu at (203.2, 112.7)
- added MX7-0: F7, MX_Alps_Hybrid:MX-1U-NoLED, F.Cu at (222.2, 112.7)
- added MX8-0: F8, MX_Alps_Hybrid:MX-1U-NoLED, F.Cu at (241.3, 112.7)
- added MX9-0: F9, MX_Alps_Hybrid:MX-1U-NoLED, F.Cu at (260.4, 112.7)
- D1, D2, D3, D4: moved to B.Cu
- MX0-0: renamed from MX1; value MX-NoLED -> Esc
- MX0-1: renamed from MX3; value MX-NoLED -> F1
- MX1-0: renamed from MX2; value MX-NoLED -> Tilde
- MX1-1: renamed from MX4; value MX-NoLED -> 1
- moved C5 30.0 mm to (60.3, 121.3)
- moved D2 26.9 mm to (96.8, 131.8)
- moved D3 26.9 mm to (115.9, 112.7)
- moved MX0-1 26.9 mm to (108.0, 112.7)
- moved MX1-0 26.9 mm to (88.9, 131.8)
- moved USB1 21.7 mm to (55.9, 106.4)
- moved C4 20.9 mm to (69.3, 142.2)
- moved C7 20.9 mm to (76.5, 133.0)
- moved R3 20.9 mm to (74.2, 123.3)
- moved U1 20.9 mm to (64.3, 132.4)
- moved Y1 20.9 mm to (64.3, 121.4)
- moved C2 20.9 mm to (69.9, 121.4)
- moved C6 20.9 mm to (67.7, 118.2)
- moved F1 20.9 mm to (64.5, 113.6)
- moved R4 20.9 mm to (55.1, 139.1)
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Connections:
- U1 pad 25: Net-(U1-Pad25) -> ROW0
- U1 pad 26: Net-(U1-Pad26) -> ROW1
- U1 pad 27: Net-(U1-Pad27) -> ROW2
- U1 pad 28: Net-(U1-Pad28) -> ROW3
- U1 pad 29: Net-(U1-Pad29) -> ROW5
- U1 pad 31: Net-(U1-Pad31) -> ROW4
- Y1 pad 2: Net-(Y1-Pad2) -> GND
Routing:
- net ROW5: track 0.00 -> 397.3 mm, vias 0 -> 1
- net ROW4: track 0.00 -> 383.2 mm, vias 0 -> 1
- net ROW0: track 0.00 -> 381.1 mm, vias 0 -> 1
- net ROW3: track 0.00 -> 376.5 mm, vias 0 -> 1
- net ROW1: track 0.00 -> 363.4 mm, vias 0 -> 1
- net ROW2: track 0.00 -> 356.9 mm, vias 0 -> 1
- net GND: track 0.00 -> 126.3 mm, vias 0 -> 4
- net COL13: track 0.00 -> 106.8 mm
- net COL2: track 0.00 -> 106.1 mm
- net COL14: track 0.00 -> 103.2 mm
- net COL0: track 0.00 -> 102.3 mm
- net COL1: track 0.00 -> 101.2 mm
- net +5V: track 0.00 -> 99.1 mm, vias 0 -> 5
- net COL12: track 0.00 -> 95.4 mm
- net COL15: track 0.00 -> 95.3 mm
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Other:
- board size 161.9 x 58.7 mm -> 335 x 114.3 mm
- net class Default: trace_width 0.25 -> 0.254
- net class power added: clearance 0.2, trace_width 0.381, via_dia 0.8, via_drill 0.4
- board text added: "1"
- board text added: "Bagnaram's Mechanical KB"
- board text added: "Matt Bagnara"

Commit message: Add gerbers
Parts:
- added REF**: OSHW-Logo2_14.6x12mm_SilkScreen, Symbol:OSHW-Logo2_14.6x12mm_SilkScreen, F.Cu at (63.5, 208.8)
- MX5-6: footprint MX_Alps_Hybrid:MX-6U-NoLED -> MX_Alps_Hybrid:MX-6U-ReversedStabilizers-NoLED
Connections:
- U1 pad 1: Net-(U1-Pad1) -> COL7
- U1 pad 12: Net-(U1-Pad12) -> COL9
- U1 pad 18: Net-(U1-Pad18) -> COL10
- U1 pad 19: Net-(U1-Pad19) -> COL11
- U1 pad 20: Net-(U1-Pad20) -> COL12
- U1 pad 21: Net-(U1-Pad21) -> COL13
- U1 pad 22: Net-(U1-Pad22) -> COL14
- U1 pad 32: Net-(U1-Pad32) -> COL15
- U1 pad 36: Net-(U1-Pad36) -> COL6
- U1 pad 37: Net-(U1-Pad37) -> COL5
- U1 pad 38: Net-(U1-Pad38) -> COL4
- U1 pad 39: Net-(U1-Pad39) -> COL3
- U1 pad 40: Net-(U1-Pad40) -> COL2
- U1 pad 41: Net-(U1-Pad41) -> COL1
- U1 pad 42: Net-(U1-Pad42) -> COL0
- U1 pad 8: Net-(U1-Pad8) -> COL8
Routing:
- net COL15: track 95.3 -> 412.1 mm, vias 0 -> 6
- net COL14: track 103.2 -> 416.5 mm, vias 0 -> 1
- net COL13: track 106.8 -> 397.4 mm, vias 0 -> 1
- net COL12: track 95.4 -> 383.2 mm, vias 0 -> 1
- net COL11: track 86.3 -> 353.8 mm, vias 0 -> 1
- net COL10: track 89.3 -> 336.5 mm, vias 0 -> 1
- net COL9: track 67.2 -> 279.9 mm, vias 0 -> 3
- net COL8: track 67.0 -> 254.7 mm, vias 0 -> 4
- net COL6: track 88.0 -> 273.9 mm, vias 0 -> 2
- net COL7: track 67.0 -> 234.3 mm, vias 0 -> 6
- net COL5: track 83.3 -> 230.1 mm, vias 0 -> 2
- net COL4: track 83.1 -> 208.6 mm, vias 0 -> 2
- net COL3: track 84.2 -> 209.0 mm, vias 0 -> 2
- net COL2: track 106.1 -> 199.7 mm, vias 0 -> 1
- net COL1: track 101.2 -> 160.6 mm, vias 0 -> 2
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Other:
- board text added: "MX Keyboard"
- board text added: "bagnaram"

Commit message: Redesign keyboard with %75 keys
Parts:
- removed D12, D18, D23, D28, D3, D33, D39, D44, D49, D54, D60, D66, D71, D72, D77, D83, D84: D_Small, Diode_SMD:D_SOD-123
- removed the MX0-1 at (108.0, 112.7)
- removed the MX0-2 at (127.0, 112.7)
- removed the MX0-3 at (146.1, 112.7)
- removed the MX0-4 at (165.1, 112.7)
- removed MX0-5: F5, MX_Alps_Hybrid:MX-1U-NoLED
- removed the MX10-0 at (279.4, 112.7)
- removed the MX11-0 at (298.4, 112.7)
- removed the MX12-0 at (317.5, 112.7)
- removed the MX13-0 at (336.6, 112.7)
- removed MX14-0: Scroll Lock, MX_Alps_Hybrid:MX-1U-NoLED
- removed MX3-15: Home, MX_Alps_Hybrid:MX-1U-NoLED
- removed MX4-14: End, MX_Alps_Hybrid:MX-1U-NoLED
- removed MX5-11: RCtrl, MX_Alps_Hybrid:MX-1U-NoLED
- removed the MX6-0 at (203.2, 112.7)
- removed the MX7-0 at (222.2, 112.7)
- removed the MX8-0 at (241.3, 112.7)
- removed the MX9-0 at (260.4, 112.7)
- removed REF**: OSHW-Logo2_14.6x12mm_SilkScreen, Symbol:OSHW-Logo2_14.6x12mm_SilkScreen
- C4: value 0.1uF -> 10uF
- MX10-4: renamed from MX5-9; value RMeta -> Fn
- MX11-4: renamed from MX5-10; value Menu -> Alt; footprint MX_Alps_Hybrid:MX-1U-NoLED -> MX_Alps_Hybrid:MX-1.25U-NoLED
- MX6-4: renamed from MX5-6; footprint MX_Alps_Hybrid:MX-6U-ReversedStabilizers-NoLED -> MX_Alps_Hybrid:MX-6.5U-ReversedStabilizers-NoLED
- moved C3 323.5 mm to (377.8, 106.4), turned to 0 degrees
- moved R4 318.5 mm to (373.1, 119.9)
- moved C4 309.6 mm to (377.8, 115.9), turned to 0 degrees
- moved C1 307.2 mm to (359.5, 108.7), turned to 180 degrees
- moved U1 304.7 mm to (368.3, 111.1), turned to -90 degrees
- moved C2 303.1 mm to (372.4, 103.4), turned to 0 degrees
- moved C5 288.3 mm to (348.3, 107.8)
- moved Y1 287.5 mm to (351.5, 107.8)
- moved C6 287.3 mm to (354.8, 107.8), turned to 90 degrees
- moved R2 286.8 mm to (342.5, 105.6), turned to 0 degrees
- moved D2 285.8 mm to (382.6, 131.8)
- moved MX15-0 285.8 mm to (374.6, 131.8)
- moved R3 285.7 mm to (359.4, 106.7), turned to 0 degrees
- moved R1 284.9 mm to (342.5, 103.3), turned to 0 degrees
- moved C7 284.3 mm to (359.4, 104.4), turned to 180 degrees
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- renumbered MX2-0 to MX0-1, MX3-0 to MX0-2, MX4-0 to MX0-3, MX5-0 to MX0-4, MX1-1 to MX1-0, MX2-1 to MX1-1, MX3-1 to MX1-2, MX5-1 to MX1-4, MX1-10 to MX10-0, MX2-10 to MX10-1, MX3-10 to MX10-2, MX4-10 to MX10-3, MX1-11 to MX11-0, MX2-11 to MX11-1, MX3-11 to MX11-2, MX4-11 to MX11-3, MX1-12 to MX12-0, MX2-12 to MX12-1, MX3-12 to MX12-2, MX4-12 to MX12-3, MX1-13 to MX13-0, MX2-13 to MX13-1, MX5-12 to MX13-4, MX4-13 to MX14,3, MX5-13 to MX14-4, MX1-0 to MX15-0, MX15-0 to MX15-1, MX1-15 to MX15-2, MX2-15 to MX15-3, MX5-14 to MX15-4, MX1-2 to MX2-0, MX2-2 to MX2-1, MX3-2 to MX2-2, MX4-2 to MX2-3, MX5-2 to MX2-4, MX1-3 to MX3-0, MX2-3 to MX3-1, MX3-3 to MX3-2, MX4-3 to MX3-3, MX1-4 to MX4-0, MX2-4 to MX4-1, MX3-4 to MX4-2, MX4-4 to MX4-3, MX1-5 to MX5-0, MX2-5 to MX5-1, MX3-5 to MX5-2, MX4-5 to MX5-3, MX1-6 to MX6-0, MX2-6 to MX6-1, MX3-6 to MX6-2, MX4-6 to MX6-3, MX1-7 to MX7-0, MX2-7 to MX7-1, MX3-7 to MX7-2, MX4-7 to MX7-3, MX1-8 to MX8-0, MX2-8 to MX8-1, MX3-8 to MX8-2, MX4-8 to MX8-3, MX1-9 to MX9-0, MX2-9 to MX9-1, MX3-9 to MX9-2, MX4-9 to MX9-3
Connections:
- net COL1 renamed /COL1
- net COL10 renamed /COL10
- net COL11 renamed /COL11
- net COL12 renamed /COL12
- net COL13 renamed /COL13
- net COL14 renamed /COL14
- net COL2 renamed /COL2
- net COL3 renamed /COL3
- net COL4 renamed /COL4
- net COL5 renamed /COL5
- net COL6 renamed /COL6
- net COL7 renamed /COL7
- net COL8 renamed /COL8
- net COL9 renamed /COL9
- net D+ renamed /D+
- net D- renamed /D-
- D1 pad 1: ROW0 -> /ROW0
- D10 pad 1: ROW3 -> /ROW3
- D11 pad 1: ROW5 -> /ROW5
- D13 pad 1: ROW1 -> /ROW0
- D14 pad 1: ROW2 -> /ROW1
- D15 pad 1: ROW3 -> /ROW3
- D16 pad 1: ROW4 -> /ROW4
- D17 pad 1: ROW5 -> /ROW5
- D19 pad 1: ROW1 -> /ROW0
- D2 pad 1: ROW1 -> /ROW0
- D20 pad 1: ROW2 -> /ROW1
- D21 pad 1: ROW3 -> /ROW3
- D22 pad 1: ROW4 -> /ROW4
- D24 pad 1: ROW1 -> /ROW0
- D25 pad 1: ROW2 -> /ROW1
- D26 pad 1: ROW3 -> /ROW3
- D27 pad 1: ROW4 -> /ROW4
- D29 pad 1: ROW1 -> /ROW0
- D30 pad 1: ROW2 -> /ROW1
- D31 pad 1: ROW3 -> /ROW3
- D32 pad 1: ROW4 -> /ROW4
- D34 pad 1: ROW1 -> /ROW0
- D35 pad 1: ROW2 -> /ROW1
- D36 pad 1: ROW3 -> /ROW3
- D37 pad 1: ROW4 -> /ROW4
- D38 pad 1: ROW5 -> /ROW5
- D4 pad 1: ROW1 -> /ROW0
- D40 pad 1: ROW1 -> /ROW0
- D41 pad 1: ROW2 -> /ROW1
- D42 pad 1: ROW3 -> /ROW3
- D43 pad 1: ROW4 -> /ROW4
- D45 pad 1: ROW1 -> /ROW0
- D46 pad 1: ROW2 -> /ROW1
- D47 pad 1: ROW3 -> /ROW3
- D48 pad 1: ROW4 -> /ROW4
- D5 pad 1: ROW2 -> /ROW1
- D50 pad 1: ROW1 -> /ROW0
- D51 pad 1: ROW2 -> /ROW1
- D52 pad 1: ROW3 -> /ROW3
- D53 pad 1: ROW4 -> /ROW4
- D55 pad 1: ROW1 -> /ROW0
- D56 pad 1: ROW2 -> /ROW1
- D57 pad 1: ROW3 -> /ROW3
- D58 pad 1: ROW4 -> /ROW4
- D59 pad 1: ROW5 -> /ROW5
- D6 pad 1: ROW3 -> /ROW3
- D61 pad 1: ROW1 -> /ROW0
- D62 pad 1: ROW2 -> /ROW1
- D63 pad 1: ROW3 -> /ROW3
- D64 pad 1: ROW4 -> /ROW4
- D65 pad 1: ROW5 -> /ROW5
- D67 pad 1: ROW1 -> /ROW0
- D68 pad 1: ROW2 -> /ROW1
- D69 pad 1: ROW3 -> /ROW3
- D7 pad 1: ROW4 -> /ROW4
- D70 pad 1: ROW4 -> /ROW4
- D73 pad 1: ROW1 -> /ROW0
- D74 pad 1: ROW2 -> /ROW1
- D76 pad 1: ROW5 -> /ROW5
- D78 pad 1: ROW4 -> /ROW4
- D79 pad 1: ROW5 -> /ROW5
- D8 pad 1: ROW5 -> /ROW5
- D80 pad 1: ROW0 -> /ROW1
- D81 pad 1: ROW1 -> /ROW3
- D82 pad 1: ROW2 -> /ROW4
- D85 pad 1: ROW5 -> /ROW5
- D9 pad 1: ROW2 -> /ROW1
- MX0-0 pad 1: COL0 -> /COL0
- MX0-1 pad 1: COL0 -> /COL0
- MX0-2 pad 1: COL0 -> /COL0
- MX0-3 pad 1: COL0 -> /COL0
- MX0-4 pad 1: COL0 -> /COL0
- MX15-0 pad 1: COL0 -> /COL15
- MX15-1 pad 1: COL15 -> /COL15
- MX15-2 pad 1: COL15 -> /COL15
- MX15-3 pad 1: COL15 -> /COL15
- MX15-4 pad 1: COL15 -> /COL15
- U1 pad 25: ROW0 -> /ROW0
- U1 pad 26: ROW1 -> /ROW1
- U1 pad 27: ROW2 -> /ROW3
- U1 pad 28: ROW3 -> /ROW4
- U1 pad 29: ROW5 -> Net-(U1-Pad29)
- U1 pad 31: ROW4 -> /ROW5
- U1 pad 32: COL15 -> /COL15
- U1 pad 42: COL0 -> /COL0
- USB1 pad 6: Net-(USB1-Pad6) -> GND
Routing:
- net COL15: track 412.1 -> 0.00 mm, vias 6 -> 0
- net ROW5: track 397.3 -> 0.00 mm, vias 1 -> 0
- net /ROW5: track 0.00 -> 385.2 mm, vias 0 -> 3
- net ROW4: track 383.2 -> 0.00 mm, vias 1 -> 0
- net /COL0: track 0.00 -> 381.1 mm, vias 0 -> 2
- net ROW0: track 381.1 -> 0.00 mm, vias 1 -> 0
- net ROW3: track 376.5 -> 0.00 mm, vias 1 -> 0
- net ROW1: track 363.4 -> 0.00 mm, vias 1 -> 0
- net ROW2: track 356.9 -> 0.00 mm, vias 1 -> 0
- net /ROW4: track 0.00 -> 356.4 mm, vias 0 -> 1
- net /ROW3: track 0.00 -> 342.1 mm, vias 0 -> 1
- net /ROW1: track 0.00 -> 327.0 mm, vias 0 -> 1
- net /COL14: track 416.5 -> 95.1 mm, vias 1 -> 0
- net /ROW0: track 0.00 -> 311.2 mm, vias 0 -> 1
- net /COL13: track 397.4 -> 109.3 mm, vias 1 -> 0
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- added copper zone on F.Cu, net GND
Other:
- board size 335 x 114.3 mm -> 304.8 x 115.9 mm
- net class Default removed
- net class power removed

Commit message: optimizations, footprint change
Parts:
- removed USB1: Molex-0548190589, Random Keyboard Parts:Molex-0548190589
- added D86: 3.6V, Diode_SMD:D_SOD-123, F.Cu at (288.9, 106.4)
- added D87: 3.6V, Diode_SMD:D_SOD-123, F.Cu at (286.5, 106.4)
- added R5: 5.1k, Resistor_SMD:R_0805_2012Metric, F.Cu at (270.3, 108.2)
- added R6: 5.1k, Resistor_SMD:R_0805_2012Metric, F.Cu at (277.4, 112.5)
- added R7: 1.5k, Resistor_SMD:R_0805_2012Metric, F.Cu at (283.7, 110.0)
- added REF**: MountingHole_2.2mm_M2_Pad, cftkb:MountingHole_2.2mm_M2_Pad, F.Cu at (83.3, 105.6)
- added REF**: MountingHole_2.2mm_M2_Pad, cftkb:MountingHole_2.2mm_M2_Pad, F.Cu at (83.3, 118.3)
- added REF**: MountingHole_2.2mm_M2_Pad, cftkb:MountingHole_2.2mm_M2_Pad, F.Cu at (231.0, 213.5)
- added REF**: MountingHole_2.2mm_M2_Pad, cftkb:MountingHole_2.2mm_M2_Pad, F.Cu at (380.2, 213.5)
- added REF**: MountingHole_2.2mm_M2_Pad, cftkb:MountingHole_2.2mm_M2_Pad, F.Cu at (380.2, 105.6)
- added REF**: MountingHole_2.2mm_M2_Pad, cftkb:MountingHole_2.2mm_M2_Pad, F.Cu at (380.2, 118.3)
- added REF**: MountingHole_2.2mm_M2_Pad, cftkb:MountingHole_2.2mm_M2_Pad, F.Cu at (231.8, 105.6)
- added REF**: MountingHole_2.2mm_M2_Pad, cftkb:MountingHole_2.2mm_M2_Pad, F.Cu at (231.8, 118.3)
- added REF**: MountingHole_2.2mm_M2_Pad, cftkb:MountingHole_2.2mm_M2_Pad, F.Cu at (83.3, 213.5)
- added SYM1: Symbol_CreativeCommons_CopperTop_Type2_Small, Symbol:Symbol_CreativeCommons_CopperTop_Type2_Small, F.Cu at (245.8, 112.0)
- added SYM2: Symbol_CC-Attribution_CopperTop_Small, Symbol:Symbol_CC-Attribution_CopperTop_Small, F.Cu at (253.2, 111.9)
- added SYM3: Symbol_CC-ShareAlike_CopperTop_Small, Symbol:Symbol_CC-ShareAlike_CopperTop_Small, F.Cu at (260.4, 111.9)
- added SYM4: OSHW-Logo2_14.6x12mm_SilkScreen, Symbol:OSHW-Logo2_14.6x12mm_SilkScreen, F.Cu at (143.7, 108.7)
- added SYM5: KiCad-Logo_5mm_SilkScreen, Symbol:KiCad-Logo_5mm_SilkScreen, F.Cu at (127.8, 108.7)
- added USB2: USB_C_GCT_USB4085-Type-C, cftkb:USB_C_GCT_USB4085, F.Cu at (277.0, 104.8)
- F1: footprint Fuse:Fuse_1206_3216Metric -> cftkb:polyfuse_5.1mm
- J1: footprint Connector_PinHeader_1.00mm:PinHeader_2x03_P1.00mm_Horizontal -> cftkb:AVR_ICSP_3x2
- MX6-4: footprint MX_Alps_Hybrid:MX-6.5U-ReversedStabilizers-NoLED -> MX_Alps_Hybrid:MX-6.25U-ReversedStabilizers-NoLED
- R1, R2: value 22 -> 75
- moved F1 41.8 mm to (287.8, 114.0), turned to 180 degrees
- moved J1 5.47 mm to (317.5, 108.0), turned to 180 degrees
- moved MX10-4 4.76 mm to (281.8, 208.0)
- moved MX11-4 4.76 mm to (305.6, 208.0)
- moved D59 3.91 mm to (290.6, 208.0)
- moved D65 3.84 mm to (314.5, 208.0)
- moved MX6-4 2.38 mm to (210.3, 208.0)
- moved C3 2.15 mm to (376.2, 105.0), turned to 90 degrees
- moved C4 1.59 mm to (378.0, 114.3)
- moved R2 0.41 mm to (342.5, 105.2)
- moved R4 0.15 mm to (373.1, 119.7)
- renumbered MX14,3 to MX14-3
Connections:
- F1 pad 1: VCC -> +5V
- F1 pad 2: +5V -> VCC
Routing:
- net /D-: track 23.3 -> 103.2 mm, vias 0 -> 2
- net /D+: track 23.3 -> 85.3 mm
- net /COL3: track 361.9 -> 307.3 mm, vias 4 -> 2
- net +5V: track 109.5 -> 146.1 mm, vias 7 -> 6
- net Net-(J1-Pad1): track 71.6 -> 47.7 mm
- net GND: track 71.1 -> 91.6 mm, vias 0 -> 6
- net VCC: track 3.06 -> 16.2 mm
- net Net-(J1-Pad3): track 59.5 -> 50.5 mm
- net (no net): track 7.73 -> 0.00 mm
- net Net-(R5-Pad1): track 0.00 -> 5.34 mm
- net /COL10: track 182.9 -> 177.7 mm
- net /ROW0: track 311.2 -> 316.0 mm
- net /ROW4: track 356.4 -> 360.2 mm
- net /ROW3: track 342.1 -> 345.9 mm
- net Net-(J1-Pad4): track 56.6 -> 60.2 mm
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Other:
- board text added: "Splendens"
- board text added: "by bagnaram"
- board text removed: "MX Keyboard"
- board text removed: "bagnaram"

Commit message: image and fixup
Parts:
- added G***: LOGO, cftkb:DISCIPLINE_SMALL_MASK, F.Cu at (189.7, 108.7)
Other:
- board text added: "Bagnaram"
- board text removed: "Bagnaram's Mechanical KB"
- board text removed: "Matt Bagnara"

Commit message: pcb image
Parts:
- renumbered J1 to ISP1
Changed lines of the file:
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@@
     (property "Sheet file" "/Users/mbagnara/Documents/my-keyboard/my-keyboard.kicad_sch")
     (property "Sheet name" "")
-    (fp_text reference "J1" (at 2.3 -1.5) (layer "F.SilkS")
+    (fp_text reference "ISP1" (at 0 -3.96875) (layer "F.SilkS")
       (effects (font (size 1 1) (thickness 0.15)))
     )

Commit message: cleanup
Parts:
- moved REF** 44.2 mm to (125.4, 200.0)
- moved REF** 40.5 mm to (342.9, 197.6)
- moved REF** 9.53 mm to (231.0, 204.0)
Changed lines of the file:
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@@
   )
   (module "cftkb:MountingHole_2.2mm_M2_Pad" (layer "F.Cu")
-    (at 230.98125 213.51875)
+    (at 230.98125 203.99375)
     (descr "Mounting Hole 2.2mm, M2")
     (tags "mounting hole 2.2mm m2")
@@
   )
   (module "cftkb:MountingHole_2.2mm_M2_Pad" (layer "F.Cu")
-    (at 380.20625 213.51875)
+    (at 342.9 197.64375)
     (descr "Mounting Hole 2.2mm, M2")
     (tags "mounting hole 2.2mm m2")
@@
     (fp_circle (center 0 0) (end 2.2 0) (layer "Cmts.User") (width 0.15))
     (fp_circle (center 0 0) (end 2.45 0) (layer "F.CrtYd") (width 0.05))
-    (pad "1" thru_hole circle (at 0 0) (size 4.4 4.4) (drill 2.2) (layers *.Cu *.Mask) (remove_unused_layers) (keep_end_layers))
+    (pad "1" thru_hole circle (at 0 0) (size 4.4 4.4) (drill 2.2) (layers *.Cu *.Mask))
   )
   (module "cftkb:MountingHole_2.2mm_M2_Pad" (layer "F.Cu")
@@
   )
   (module "cftkb:MountingHole_2.2mm_M2_Pad" (layer "F.Cu")
-    (at 83.34375 213.51875)
+    (at 125.4125 200.025)
     (descr "Mounting Hole 2.2mm, M2")
     (tags "mounting hole 2.2mm m2")
