File: my-keyboard.kicad_pcb (KiCad board)
At the start: 2 copper layers, 304.8 x 115.9 mm, 171 parts, among them SW1 SW_Push, U1 ATmega32U4-AU, Y1 16MHz

Commit message: Generated gerbers
Parts:
- C1, C2, C3: value 0.1uF -> 0.1u
- C4: value 10uF -> 10u
- C5, C6: value 22pF -> 22p
- C7: value 1uF -> 1u
- R1, R2: value 75 -> 22
- USB1: value USB_C_GCT_USB4085-Type-C -> Wurth-632723300011; footprint SnapEDA:AMPHENOL_10137061-00021LF -> Type-C:Wurth-632723300011
- moved R6 12.5 mm to (282.2, 106.2), turned to -90 degrees
- moved C2 12.2 mm to (378.0, 114.3)
- moved C4 12.2 mm to (372.6, 103.4)
- moved USB1 10.3 mm to (276.2, 100.0)
Routing:
- net VCC: track 11.7 -> 27.0 mm
- net GND: track 84.9 -> 74.7 mm
- net /D-: track 94.6 -> 87.9 mm
- net Net-(R6-Pad2): track 6.81 -> 10.7 mm, vias 2 -> 0
Other:
- board text added: "Ocotillo"

Commit message: fix aref pin
Connections:
- U1 pad 29: Net-(U1-Pad29) -> /COL0
- U1 pad 42: /COL0 -> Net-(U1-Pad42)
Routing:
- net /COL0: track 384.4 -> 379.7 mm
Other:
- board text added: "1.1"
- board text removed: "1"
- board text removed: "Splendens"
Changed lines of the file:
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@@
   (net 102 "/D-")
   (net 103 "/D+")
-  (net 104 "Net-(U1-Pad29)")
+  (net 104 "Net-(U1-Pad42)")
   (net 105 "Net-(R5-Pad1)")
   (net 106 "VCC")
@@
     (property "Sheet name" "")
     (attr smd)
-    (fp_text reference "R3" (at -2.794 -2.54) (layer "F.SilkS")
+    (fp_text reference "R3" (at -2.794 0) (layer "F.SilkS")
       (effects (font (size 1 1) (thickness 0.15)))
     )
@@
       (net 12 "/ROW4") (pinfunction "PB4"))
     (pad "29" smd rect (at 5.7 -0.8 270) (size 1.5 0.55) (layers "F.Cu" "F.Paste" "F.Mask")
-      (net 104 "Net-(U1-Pad29)") (pinfunction "PB5"))
+      (net 20 "/COL0") (pinfunction "PB5"))
     (pad "30" smd rect (at 5.7 -1.6 270) (size 1.5 0.55) (layers "F.Cu" "F.Paste" "F.Mask")
       (net 18 "Net-(U1-Pad30)") (pinfunction "PB6"))
@@
       (net 22 "/COL1") (pinfunction "PF0"))
     (pad "42" smd rect (at -2.4 -5.7) (size 1.5 0.55) (layers "F.Cu" "F.Paste" "F.Mask")
-      (net 20 "/COL0") (pinfunction "AREF"))
+      (net 104 "Net-(U1-Pad42)") (pinfunction "AREF"))
     (pad "43" smd rect (at -3.2 -5.7) (size 1.5 0.55) (layers "F.Cu" "F.Paste" "F.Mask")
       (net 1 "GND") (pinfunction "GND"))
@@
     )
   )
-  (module "Crystal:Crystal_SMD_3225-4Pin_3.2x2.5mm" (layer "F.Cu")
+  (module "Crystal:Crystal_SMD_3225-4Pin_3.2x2.5mm" locked (layer "F.Cu")
     (at 351.493 107.784)
     (descr "SMD Crystal SERIES SMD3225/4 http://www.txccrystal.com/images/pdf/7m-accuracy.pdf, 3.2x2.5mm^2 package")
@@
     (property "Sheet name" "")
     (attr smd)
-    (fp_text reference "C7" (at 2.54 -3.048 180) (layer "F.SilkS")
+    (fp_text reference "C7" (at 3.048 0 180) (layer "F.SilkS")
       (effects (font (size 1 1) (thickness 0.15)))
     )
@@
   (gr_arc (start 382.5875 103.1875) (end 384.175 103.1875) (angle -90) (layer "Edge.Cuts") (width 0.05))
   (gr_arc (start 382.5875 215.9) (end 382.5875 217.4875) (angle -90) (layer "Edge.Cuts") (width 0.05))
-  (gr_text "1" (at 392.1125 280.19375) (layer "F.Cu")
+  (gr_text "1.1" (at 393.192 280.19375) (layer "F.Cu")
     (effects (font (size 1.5 1.5) (thickness 0.3)))
   )
@@
     (effects (font (size 3 3) (thickness 0.3)))
   )
-  (gr_text "Splendens" (at 315.9125 276.225) (layer "F.Cu")
+  (gr_text "Ocotillo" (at 315.9125 276.225) (layer "F.Cu")
     (effects (font (size 1.5 1.5) (thickness 0.3)))
   )
@@
   (segment (start 98.75 146.3125) (end 101.6 149.1625) (width 0.254) (layer "B.Cu") (net 19))
   (segment (start 96.1625 146.3125) (end 98.75 146.3125) (width 0.254) (layer "B.Cu") (net 19))
-  (segment (start 372.364 108.712) (end 373.987 108.712) (width 0.254) (layer "F.Cu") (net 20))
   (segment (start 90.5025 164.20125) (end 92.88375 166.5825) (width 0.254) (layer "F.Cu") (net 20))
   (segment (start 85.74 142.77) (end 90.5025 147.5325) (width 0.254) (layer "F.Cu") (net 20))
   (segment (start 100.10453 114.20797) (end 233.736168 114.20797) (width 0.254) (layer "F.Cu") (net 20))
-  (segment (start 334.61003 115.98597) (end 342.138 108.458) (width 0.254) (layer "F.Cu") (net 20))
+  (segment (start 369.062 116.787) (end 369.1 116.825) (width 0.254) (layer "F.Cu") (net 20))
   (segment (start 97.64625 185.6325) (end 97.64625 195.1575) (width 0.254) (layer "F.Cu") (net 20))
+  (segment (start 369.062 115.316) (end 369.062 116.787) (width 0.254) (layer "F.Cu") (net 20))
   (segment (start 90.5025 147.5325) (end 90.5025 164.20125) (width 0.254) (layer "F.Cu") (net 20))
   (segment (start 233.736168 114.20797) (end 235.514168 115.98597) (width 0.254) (layer "F.Cu") (net 20))
   (segment (start 235.514168 115.98597) (end 334.61003 115.98597) (width 0.254) (layer "F.Cu") (net 20))
   (segment (start 92.88375 166.5825) (end 92.88375 180.87) (width 0.254) (layer "F.Cu") (net 20))
+  (segment (start 334.86403 115.98597) (end 335.28 115.57) (width 0.254) (layer "F.Cu") (net 20))
+  (segment (start 334.61003 115.98597) (end 334.86403 115.98597) (width 0.254) (layer "F.Cu") (net 20))
   (segment (start 92.88375 180.87) (end 97.64625 185.6325) (width 0.254) (layer "F.Cu") (net 20))
   (segment (start 97.64625 195.1575) (end 88.12125 204.6825) (width 0.254) (layer "F.Cu") (net 20))
   (segment (start 85.09 129.2225) (end 100.10453 114.20797) (width 0.254) (layer "F.Cu") (net 20))
   (segment (start 85.74 128.4825) (end 85.74 142.77) (width 0.254) (layer "F.Cu") (net 20))
-  (via (at 342.138 108.458) (size 0.8) (drill 0.4) (layers "F.Cu" "B.Cu") (net 20))
-  (via (at 372.618 108.712) (size 0.8) (drill 0.4) (layers "F.Cu" "B.Cu") (net 20))
-  (segment (start 342.138 108.458) (end 372.364 108.458) (width 0.254) (layer "B.Cu") (net 20))
-  (segment (start 372.364 108.458) (end 372.618 108.712) (width 0.254) (layer "B.Cu") (net 20))
+  (via (at 369.062 115.316) (size 0.8) (drill 0.4) (layers "F.Cu" "B.Cu") (net 20))
+  (via (at 335.28 115.57) (size 0.8) (drill 0.4) (layers "F.Cu" "B.Cu") (net 20))
+  (segment (start 337.525514 117.815514) (end 366.562486 117.815514) (width 0.254) (layer "B.Cu") (net 20))
+  (segment (start 366.562486 117.815514) (end 369.062 115.316) (width 0.254) (layer "B.Cu") (net 20))
+  (segment (start 335.28 115.57) (end 337.525514 117.815514) (width 0.254) (layer "B.Cu") (net 20))
   (segment (start 98.58375 164.7825) (end 100.55125 164.7825) (width 0.254) (layer "B.Cu") (net 21))
   (segment (start 100.55125 164.7825) (end 103.98125 168.2125) (width 0.254) (layer "B.Cu") (net 21))
